File: v3/analog_sensors.kicad_sch (KiCad schematic)
At the start: 12 parts, among them M1 JST A1, M1 JST A2, M1 JST A3, M1 JST A4

Commit message: first iteration ready for review
Parts:
- removed GND: A2, TestPoint:TestPoint_Pad_D1.0mm, symbol Connector:TestPoint
- removed GND: A3, TestPoint:TestPoint_Pad_D1.0mm, symbol Connector:TestPoint
- removed GND: A4, TestPoint:TestPoint_Pad_D1.0mm, symbol Connector:TestPoint
- removed GND: A1, TestPoint:TestPoint_Pad_D1.0mm, symbol Connector:TestPoint
Changed lines of the file:
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@@
   (junction (at 185.42 36.83) (diameter 0) (color 0 0 0 0)
   )
-  (junction (at 31.75 41.91) (diameter 0) (color 0 0 0 0)
-  )
-  (junction (at 185.42 41.91) (diameter 0) (color 0 0 0 0)
-  )
   (junction (at 82.55 36.83) (diameter 0) (color 0 0 0 0)
   )
   (junction (at 133.35 36.83) (diameter 0) (color 0 0 0 0)
   )
-  (junction (at 82.55 41.91) (diameter 0) (color 0 0 0 0)
-  )
   (junction (at 31.75 36.83) (diameter 0) (color 0 0 0 0)
-  )
-  (junction (at 133.35 41.91) (diameter 0) (color 0 0 0 0)
   )
   (no_connect (at 69.85 36.83))
@@
   (no_connect (at 172.72 36.83))
   (no_connect (at 120.65 36.83))
-  (wire (pts (xy 185.42 41.91) (xy 185.42 44.45))
-    (stroke (width 0) (type default))
-  )
   (wire (pts (xy 128.27 36.83) (xy 133.35 36.83))
     (stroke (width 0) (type default))
@@
     (stroke (width 0) (type default))
   )
-  (wire (pts (xy 133.35 41.91) (xy 133.35 44.45))
-    (stroke (width 0) (type default))
-  )
-  (wire (pts (xy 185.42 36.83) (xy 185.42 41.91))
+  (wire (pts (xy 185.42 36.83) (xy 185.42 44.45))
     (stroke (width 0) (type default))
   )
@@
     (stroke (width 0) (type default))
   )
-  (wire (pts (xy 82.55 41.91) (xy 82.55 44.45))
-    (stroke (width 0) (type default))
-  )
-  (wire (pts (xy 31.75 36.83) (xy 31.75 41.91))
+  (wire (pts (xy 31.75 36.83) (xy 31.75 44.45))
     (stroke (width 0) (type default))
   )
@@
     (stroke (width 0) (type default))
   )
-  (wire (pts (xy 133.35 36.83) (xy 133.35 41.91))
-    (stroke (width 0) (type default))
-  )
-  (wire (pts (xy 82.55 36.83) (xy 82.55 41.91))
+  (wire (pts (xy 133.35 36.83) (xy 133.35 44.45))
+    (stroke (width 0) (type default))
+  )
+  (wire (pts (xy 82.55 36.83) (xy 82.55 44.45))
     (stroke (width 0) (type default))
   )
@@
   )
   (wire (pts (xy 35.56 34.29) (xy 38.1 34.29))
-    (stroke (width 0) (type default))
-  )
-  (wire (pts (xy 31.75 41.91) (xy 31.75 44.45))
     (stroke (width 0) (type default))
   )
@@
     (effects (font (size 1.27 1.27)) (justify right))
   )
-  (symbol (lib_id "Connector:TestPoint") (at 82.55 41.91 270) (unit 1)
-    (in_bom yes) (on_board yes) (dnp no)
-    (property "Reference" "GND" (at 88.9 43.18 90)
-      (effects (font (size 1.27 1.27)) (justify left))
-    )
-    (property "Value" "A2" (at 88.9 40.64 90)
-      (effects (font (size 1.27 1.27)) (justify left))
-    )
-    (property "Footprint" "TestPoint:TestPoint_Pad_D1.0mm" (at 82.55 46.99 0)
-      (effects (font (size 1.27 1.27)) hide)
-    )
-    (property "Datasheet" "~" (at 82.55 46.99 0)
-      (effects (font (size 1.27 1.27)) hide)
-    )
-    (pin "1")
-    (instances
-      (project "CollabJam"
-        (path "/9bdfecce-164d-4fcf-8d25-7676433448a3/ab1fce9d-ef64-4e01-b2d3-d6d949317aab"
-          (reference "GND") (unit 1)
-        )
-        (path "/9bdfecce-164d-4fcf-8d25-7676433448a3/e9c2f3e2-d4c0-40ac-917d-f5e903ca1042"
-          (reference "TestA2") (unit 1)
-        )
-      )
-    )
-  )
   (symbol (lib_id "Device:R_Potentiometer_Trim") (at 176.53 36.83 270) (unit 1)
     (in_bom yes) (on_board yes) (dnp no) (fields_autoplaced)
@@
         (path "/9bdfecce-164d-4fcf-8d25-7676433448a3/e9c2f3e2-d4c0-40ac-917d-f5e903ca1042"
           (reference "RV4") (unit 1)
-        )
-      )
-    )
-  )
-  (symbol (lib_id "Connector:TestPoint") (at 133.35 41.91 270) (unit 1)
-    (in_bom yes) (on_board yes) (dnp no)
-    (property "Reference" "GND" (at 139.7 43.18 90)
-      (effects (font (size 1.27 1.27)) (justify left))
-    )
-    (property "Value" "A3" (at 139.7 40.64 90)
-      (effects (font (size 1.27 1.27)) (justify left))
-    )
-    (property "Footprint" "TestPoint:TestPoint_Pad_D1.0mm" (at 133.35 46.99 0)
-      (effects (font (size 1.27 1.27)) hide)
-    )
-    (property "Datasheet" "~" (at 133.35 46.99 0)
-      (effects (font (size 1.27 1.27)) hide)
-    )
-    (pin "1")
-    (instances
-      (project "CollabJam"
-        (path "/9bdfecce-164d-4fcf-8d25-7676433448a3/ab1fce9d-ef64-4e01-b2d3-d6d949317aab"
-          (reference "GND") (unit 1)
-        )
-        (path "/9bdfecce-164d-4fcf-8d25-7676433448a3/e9c2f3e2-d4c0-40ac-917d-f5e903ca1042"
-          (reference "TestA3") (unit 1)
         )
       )
@@
         )
       )
-    )
-  )
-  (symbol (lib_id "Connector:TestPoint") (at 185.42 41.91 270) (unit 1)
-    (in_bom yes) (on_board yes) (dnp no)
-    (property "Reference" "GND" (at 191.77 43.18 90)
-      (effects (font (size 1.27 1.27)) (justify left))
-    )
-    (property "Value" "A4" (at 191.77 40.64 90)
-      (effects (font (size 1.27 1.27)) (justify left))
-    )
-    (property "Footprint" "TestPoint:TestPoint_Pad_D1.0mm" (at 185.42 46.99 0)
-      (effects (font (size 1.27 1.27)) hide)
-    )
-    (property "Datasheet" "~" (at 185.42 46.99 0)
-      (effects (font (size 1.27 1.27)) hide)
-    )
-    (pin "1")
-    (instances
-      (project "CollabJam"
-        (path "/9bdfecce-164d-4fcf-8d25-7676433448a3/ab1fce9d-ef64-4e01-b2d3-d6d949317aab"
-          (reference "GND") (unit 1)
-        )
-        (path "/9bdfecce-164d-4fcf-8d25-7676433448a3/e9c2f3e2-d4c0-40ac-917d-f5e903ca1042"
-          (reference "TestA4") (unit 1)
-        )
-      )
-    )
-  )
-  (symbol (lib_id "Connector:TestPoint") (at 31.75 41.91 270) (unit 1)
-    (in_bom yes) (on_board yes) (dnp no)
-    (property "Reference" "GND" (at 38.1 43.18 90)
-      (effects (font (size 1.27 1.27)) (justify left))
-    )
-    (property "Value" "A1" (at 38.1 40.64 90)
-      (effects (font (size 1.27 1.27)) (justify left))
-    )
-    (property "Footprint" "TestPoint:TestPoint_Pad_D1.0mm" (at 31.75 46.99 0)
-      (effects (font (size 1.27 1.27)) hide)
-    )
-    (property "Datasheet" "~" (at 31.75 46.99 0)
-      (effects (font (size 1.27 1.27)) hide)
-    )
-    (pin "1")
-    (instances
-      (project "CollabJam"
-        (path "/9bdfecce-164d-4fcf-8d25-7676433448a3/ab1fce9d-ef64-4e01-b2d3-d6d949317aab"
-          (reference "GND") (unit 1)
-        )
-        (path "/9bdfecce-164d-4fcf-8d25-7676433448a3/e9c2f3e2-d4c0-40ac-917d-f5e903ca1042"
-          (reference "TestA1") (unit 1)
-        )
-      )
