File: v4/motor_drivers-QFN.kicad_sch (KiCad schematic)
At the start: 40 parts, among them IC2 DA7282, IC3 DA7282, IC4 DA7282, IC5 DA7282, IC6 DA7282, IC7 DA7282, J2 Conn_01x16_Pin, M1 M1, M2 M2, M3 M3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

Commit message: fix bom
Parts:
- C7: value C -> 1uF
- M1, M2, M3, M4, M5, M6: now left out of the parts list
Changed lines of the file:
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@@
 		(unit 1)
 		(exclude_from_sim no)
-		(in_bom yes)
+		(in_bom no)
 		(on_board yes)
 		(dnp no)
@@
 		(unit 1)
 		(exclude_from_sim no)
-		(in_bom yes)
+		(in_bom no)
 		(on_board yes)
 		(dnp no)
@@
 		(unit 1)
 		(exclude_from_sim no)
-		(in_bom yes)
+		(in_bom no)
 		(on_board yes)
 		(dnp no)
@@
 			)
 		)
-		(property "Value" "C"
+		(property "Value" "1uF"
 			(at 236.22 21.59 90)
 			(effects
@@
 		(unit 1)
 		(exclude_from_sim no)
-		(in_bom yes)
+		(in_bom no)
 		(on_board yes)
 		(dnp no)
@@
 		(unit 1)
 		(exclude_from_sim no)
-		(in_bom yes)
+		(in_bom no)
 		(on_board yes)
 		(dnp no)
@@
 		(unit 1)
 		(exclude_from_sim no)
-		(in_bom yes)
+		(in_bom no)
 		(on_board yes)
 		(dnp no)
